Commit message: add joint limits for the double pendulum example

File: robots/double_pendulum_description/urdf/double_pendulum.urdf (robot description, URDF)
Before this commit: robot 2dof_planar, 3 links, 2 joints
Joints:
- joint joint1: limit lower=0 upper=0 effort=0 velocity=0 -> lower=2.3561945 upper=3.9269908 effort=0.8 velocity=10
- joint joint2: limit lower=0 upper=0 effort=0 velocity=0 -> lower=2.3561945 upper=3.9269908 effort=0.8 velocity=10

Commit message: more realistic joint bounds

File: robots/double_pendulum_description/urdf/double_pendulum.urdf (robot description, URDF)
Before this commit: robot 2dof_planar, 3 links, 2 joints
Joints:
- joint joint1: limit lower=2.3561945 upper=3.9269908 effort=0.8 velocity=10 -> lower=-3.9269908 upper=-2.3561945 effort=0.8 velocity=10
- joint joint2: limit lower=2.3561945 upper=3.9269908 effort=0.8 velocity=10 -> lower=-0.7853982 upper=0.7853982 effort=0.8 velocity=10

Commit message: larger position bounds for dp

File: robots/double_pendulum_description/urdf/double_pendulum.urdf (robot description, URDF)
Before this commit: robot 2dof_planar, 3 links, 2 joints
Joints:
- joint joint1: limit lower=-3.9269908 upper=-2.3561945 effort=0.8 velocity=10 -> lower=-4.7123890 upper=-1.5707963 effort=1.8 velocity=10
- joint joint2: limit lower=-0.7853982 upper=0.7853982 effort=0.8 velocity=10 -> lower=-1.5707963 upper=1.5707963 effort=1.8 velocity=10
